File: spisolator.sch (KiCad schematic (older format))
At the start: 18 parts

Commit message: annotate schematics
Parts:
- gave numbers to parts that had none: 12
Connections:
- net at U1.2 (O/I), U2.1 (~CS): now also U1.4 (I/O); no longer U1.1 (I/O)
- net at P2.1 (P1): now also U1.3 (O/I); no longer U1.2 (O/I)
- net at P2.3 (P3): now also U1.10 (O/I); no longer U1.3 (O/I)
- net at P2.8 (P8): now also U3.3 (O/I); no longer U3.9 (O/I)
- net at U2.6 (CLK), U3.11 (I/O): now also U3.9 (O/I); no longer U3.10 (O/I)
- net at P1.3 (P3): now also U1.8 (I/O); no longer U1.4 (I/O)
- net at P1.6 (P6): now also U3.8 (I/O); no longer U3.11 (I/O)
- net at P1.8 (P8): now also U3.1 (I/O); no longer U3.8 (I/O)
- new net: J1.3 (Pin_3), U1.12 (ON), U1.5 (ON), U3.12 (ON), U3.5 (ON)
- new net: U1.11 (I/O), U1.9 (O/I), U2.2 (SO)
- new net: U2.5 (SI), U3.2 (O/I), U3.4 (I/O)
- new net: J1.1 (Pin_1), U1.13 (ON), U1.6 (ON), U3.13 (ON), U3.6 (ON)

Commit message: assosiate footprints
Connections:
- no-connect marks 0 -> 4
Changed lines of the file:
@@
 $EndComp
 $Comp
-L +3.3V #PWR16
+L +3.3V #PWR01
 U 1 1 5B0F5F09
 P 6200 3750
-F 0 "#PWR16" H 6200 3600 50  0001 C CNN
+F 0 "#PWR01" H 6200 3600 50  0001 C CNN
 F 1 "+3.3V" H 6200 3890 50  0000 C CNN
 F 2 "" H 6200 3750 50  0001 C CNN
@@
 $EndComp
 $Comp
-L +3.3V #PWR3
+L +3.3V #PWR02
 U 1 1 5B0F70C6
 P 3700 3950
-F 0 "#PWR3" H 3700 3800 50  0001 C CNN
+F 0 "#PWR02" H 3700 3800 50  0001 C CNN
 F 1 "+3.3V" H 3700 4090 50  0000 C CNN
 F 2 "" H 3700 3950 50  0001 C CNN
@@
 $EndComp
 $Comp
-L GND #PWR7
+L GND #PWR03
 U 1 1 5B0F8116
 P 4700 4350
-F 0 "#PWR7" H 4700 4100 50  0001 C CNN
+F 0 "#PWR03" H 4700 4100 50  0001 C CNN
 F 1 "GND" H 4700 4200 50  0000 C CNN
 F 2 "" H 4700 4350 50  0001 C CNN
@@
 $EndComp
 $Comp
-L +3.3V #PWR13
+L +3.3V #PWR04
 U 1 1 5B0F81F9
-P 5250 5050
-F 0 "#PWR13" H 5250 4900 50  0001 C CNN
-F 1 "+3.3V" H 5250 5190 50  0000 C CNN
-F 2 "" H 5250 5050 50  0001 C CNN
-F 3 "" H 5250 5050 50  0001 C CNN
-	1    5250 5050
-	1    0    0    -1
-$EndComp
-$Comp
-L +3.3V #PWR19
+P 5350 5050
+F 0 "#PWR04" H 5350 4900 50  0001 C CNN
+F 1 "+3.3V" H 5350 5190 50  0000 C CNN
+F 2 "" H 5350 5050 50  0001 C CNN
+F 3 "" H 5350 5050 50  0001 C CNN
+	1    5350 5050
+	1    0    0    -1
+$EndComp
+$Comp
+L +3.3V #PWR05
 U 1 1 5B0F8264
 P 6350 5050
-F 0 "#PWR19" H 6350 4900 50  0001 C CNN
+F 0 "#PWR05" H 6350 4900 50  0001 C CNN
 F 1 "+3.3V" H 6350 5190 50  0000 C CNN
 F 2 "" H 6350 5050 50  0001 C CNN
@@
 $EndComp
 $Comp
-L +3.3V #PWR23
+L +3.3V #PWR06
 U 1 1 5B0F82A3
 P 7300 5050
-F 0 "#PWR23" H 7300 4900 50  0001 C CNN
+F 0 "#PWR06" H 7300 4900 50  0001 C CNN
 F 1 "+3.3V" H 7300 5190 50  0000 C CNN
 F 2 "" H 7300 5050 50  0001 C CNN
@@
 $EndComp
 $Comp
-L GND #PWR4
+L GND #PWR07
 U 1 1 5B0F8C25
 P 3700 5050
-F 0 "#PWR4" H 3700 4800 50  0001 C CNN
+F 0 "#PWR07" H 3700 4800 50  0001 C CNN
 F 1 "GND" H 3700 4900 50  0000 C CNN
 F 2 "" H 3700 5050 50  0001 C CNN
@@
 $EndComp
 $Comp
-L GND #PWR9
+L GND #PWR08
 U 1 1 5B0F8CA4
 P 4750 5050
-F 0 "#PWR9" H 4750 4800 50  0001 C CNN
+F 0 "#PWR08" H 4750 4800 50  0001 C CNN
 F 1 "GND" H 4750 4900 50  0000 C CNN
 F 2 "" H 4750 5050 50  0001 C CNN
@@
 $EndComp
 $Comp
-L GND #PWR15
+L GND #PWR09
 U 1 1 5B0F8CE3
 P 5650 5050
-F 0 "#PWR15" H 5650 4800 50  0001 C CNN
+F 0 "#PWR09" H 5650 4800 50  0001 C CNN
 F 1 "GND" H 5650 4900 50  0000 C CNN
 F 2 "" H 5650 5050 50  0001 C CNN
@@
 $EndComp
 $Comp
-L GND #PWR21
+L GND #PWR010
 U 1 1 5B0F8D15
 P 6600 5050
-F 0 "#PWR21" H 6600 4800 50  0001 C CNN
+F 0 "#PWR010" H 6600 4800 50  0001 C CNN
 F 1 "GND" H 6600 4900 50  0000 C CNN
 F 2 "" H 6600 5050 50  0001 C CNN
@@
 $EndComp
 $Comp
-L GND #PWR10
+L GND #PWR011
 U 1 1 5B0F9995
 P 4950 6350
-F 0 "#PWR10" H 4950 6100 50  0001 C CNN
+F 0 "#PWR011" H 4950 6100 50  0001 C CNN
 F 1 "GND" H 4950 6200 50  0000 C CNN
 F 2 "" H 4950 6350 50  0001 C CNN
@@
 $EndComp
 $Comp
-L +3.3V #PWR6
+L +3.3V #PWR012
 U 1 1 5B0FB499
 P 4400 5050
-F 0 "#PWR6" H 4400 4900 50  0001 C CNN
+F 0 "#PWR012" H 4400 4900 50  0001 C CNN
 F 1 "+3.3V" H 4400 5190 50  0000 C CNN
 F 2 "" H 4400 5050 50  0001 C CNN
@@
 $EndComp
 $Comp
-L +3.3V #PWR12
+L +3.3V #PWR013
 U 1 1 5B0FD818
 P 5250 2900
-F 0 "#PWR12" H 5250 2750 50  0001 C CNN
+F 0 "#PWR013" H 5250 2750 50  0001 C CNN
 F 1 "+3.3V" H 5250 3040 50  0000 C CNN
 F 2 "" H 5250 2900 50  0001 C CNN
@@
 $EndComp
 $Comp
-L +3.3V #PWR18
+L +3.3V #PWR014
 U 1 1 5B0FD81E
 P 6350 2900
-F 0 "#PWR18" H 6350 2750 50  0001 C CNN
+F 0 "#PWR014" H 6350 2750 50  0001 C CNN
 F 1 "+3.3V" H 6350 3040 50  0000 C CNN
 F 2 "" H 6350 2900 50  0001 C CNN
@@
 $EndComp
 $Comp
-L +3.3V #PWR22
+L +3.3V #PWR015
 U 1 1 5B0FD824
 P 7300 2900
-F 0 "#PWR22" H 7300 2750 50  0001 C CNN
+F 0 "#PWR015" H 7300 2750 50  0001 C CNN
 F 1 "+3.3V" H 7300 3040 50  0000 C CNN
 F 2 "" H 7300 2900 50  0001 C CNN
@@
 $EndComp
 $Comp
-L GND #PWR2
+L GND #PWR016
 U 1 1 5B0FD82A
 P 3700 2900
-F 0 "#PWR2" H 3700 2650 50  0001 C CNN
+F 0 "#PWR016" H 3700 2650 50  0001 C CNN
 F 1 "GND" H 3700 2750 50  0000 C CNN
 F 2 "" H 3700 2900 50  0001 C CNN
@@
 $EndComp
 $Comp
-L GND #PWR8
+L GND #PWR017
 U 1 1 5B0FD830
-P 4750 2900
-F 0 "#PWR8" H 4750 2650 50  0001 C CNN
-F 1 "GND" H 4750 2750 50  0000 C CNN
-F 2 "" H 4750 2900 50  0001 C CNN
-F 3 "" H 4750 2900 50  0001 C CNN
-	1    4750 2900
-	1    0    0    -1
-$EndComp
-$Comp
-L GND #PWR14
+P 4650 2900
+F 0 "#PWR017" H 4650 2650 50  0001 C CNN
+F 1 "GND" H 4650 2750 50  0000 C CNN
+F 2 "" H 4650 2900 50  0001 C CNN
+F 3 "" H 4650 2900 50  0001 C CNN
+	1    4650 2900
+	1    0    0    -1
+$EndComp
+$Comp
+L GND #PWR018
 U 1 1 5B0FD836
 P 5650 2900
-F 0 "#PWR14" H 5650 2650 50  0001 C CNN
+F 0 "#PWR018" H 5650 2650 50  0001 C CNN
 F 1 "GND" H 5650 2750 50  0000 C CNN
 F 2 "" H 5650 2900 50  0001 C CNN
@@
 $EndComp
 $Comp
-L GND #PWR20
+L GND #PWR019
 U 1 1 5B0FD83C
 P 6600 2900
-F 0 "#PWR20" H 6600 2650 50  0001 C CNN
+F 0 "#PWR019" H 6600 2650 50  0001 C CNN
 F 1 "GND" H 6600 2750 50  0000 C CNN
 F 2 "" H 6600 2900 50  0001 C CNN
@@
 $EndComp
 $Comp
-L +3.3V #PWR5
+L +3.3V #PWR020
 U 1 1 5B0FD842
 P 4400 2900
-F 0 "#PWR5" H 4400 2750 50  0001 C CNN
+F 0 "#PWR020" H 4400 2750 50  0001 C CNN
 F 1 "+3.3V" H 4400 3040 50  0000 C CNN
 F 2 "" H 4400 2900 50  0001 C CNN
@@
 $EndComp
 $Comp
-L GND #PWR11
+L GND #PWR021
 U 1 1 5B0FE734
 P 5100 1750
-F 0 "#PWR11" H 5100 1500 50  0001 C CNN
+F 0 "#PWR021" H 5100 1500 50  0001 C CNN
 F 1 "GND" H 5100 1600 50  0000 C CNN
 F 2 "" H 5100 1750 50  0001 C CNN
@@
 $EndComp
 $Comp
-L GND #PWR17
+L GND #PWR022
 U 1 1 5B100C7B
 P 6200 4200
-F 0 "#PWR17" H 6200 3950 50  0001 C CNN
+F 0 "#PWR022" H 6200 3950 50  0001 C CNN
 F 1 "GND" H 6200 4050 50  0000 C CNN
 F 2 "" H 6200 4200 50  0001 C CNN
@@
 $EndComp
 $Comp
-L GND #PWR25
+L GND #PWR023
 U 1 1 5B10383A
 P 7800 1950
-F 0 "#PWR25" H 7800 1700 50  0001 C CNN
+F 0 "#PWR023" H 7800 1700 50  0001 C CNN
 F 1 "GND" H 7800 1800 50  0000 C CNN
 F 2 "" H 7800 1950 50  0001 C CNN
@@
 $EndComp
 $Comp
-L +3.3V #PWR24
+L +3.3V #PWR024
 U 1 1 5B104C8F
 P 7800 1550
-F 0 "#PWR24" H 7800 1400 50  0001 C CNN
+F 0 "#PWR024" H 7800 1400 50  0001 C CNN
 F 1 "+3.3V" H 7800 1690 50  0000 C CNN
 F 2 "" H 7800 1550 50  0001 C CNN
@@
 VCC_Flasher
 $Comp
-L +3.3V #PWR26
+L +3.3V #PWR025
 U 1 1 5B105436
 P 8800 900
-F 0 "#PWR26" H 8800 750 50  0001 C CNN
+F 0 "#PWR025" H 8800 750 50  0001 C CNN
 F 1 "+3.3V" H 8800 1040 50  0000 C CNN
 F 2 "" H 8800 900 50  0001 C CNN
@@
 $EndComp
 $Comp
-L +3.3V #PWR1
+L +3.3V #PWR026
 U 1 1 5B10AB37
 P 3200 3400
-F 0 "#PWR1" H 3200 3250 50  0001 C CNN
+F 0 "#PWR026" H 3200 3250 50  0001 C CNN
 F 1 "+3.3V" H 3200 3540 50  0000 C CNN
 F 2 "" H 3200 3400 50  0001 C CNN
@@
 	0    1    1    0
 $EndComp
+NoConn ~ 5600 1350
+NoConn ~ 5100 1450
+NoConn ~ 5100 6250
+NoConn ~ 5600 6150
 Wire Wire Line
 	5600 4000 5700 4000
@@
 	4700 4350 4700 4200
 Wire Wire Line
-	4950 6350 5100 6350
-Wire Wire Line
 	4550 4550 5000 4550
 Wire Wire Line
@@
 	6600 5050 6700 5050
 Wire Wire Line
-	5750 5050 5650 5050
-Wire Wire Line
-	5750 5150 5650 5150
-Wire Wire Line
 	3700 5050 3800 5050
 Wire Wire Line
 	4300 5050 4400 5050
-Wire Wire Line
-	6350 5050 6250 5050
 Wire Wire Line
 	4350 3500 4350 4550
@@
 Wire Wire Line
 	3700 2900 3800 2900
-Wire Wire Line
-	4300 2900 4400 2900
 Wire Wire Line
 	6350 2900 6250 2900
@@
 Wire Wire Line
 	3200 3400 3000 3400
+Wire Wire Line
+	5250 5050 5350 5050
+Wire Wire Line
+	5100 6350 4950 6350
+Wire Wire Line
+	4300 2900 4400 2900
+Wire Wire Line
+	5750 5050 5650 5050
+Wire Wire Line
+	6250 5050 6350 5050
+Wire Wire Line
+	4650 2900 4750 2900
 $EndSCHEMATC

Commit message: schematics: add net annotations, correct logicbuffer, ...
Parts:
- C1, C2: footprint (none) -> Capacitors_SMD:C_0603_HandSoldering
- J1, J2: footprint (none) -> Pin_Headers:Pin_Header_Straight_1x03_Pitch2.54mm
- P1, P2: footprint (none) -> Pin_Headers:Pin_Header_Straight_2x04_Pitch2.54mm
- R1, R2, R3: footprint (none) -> Resistors_SMD:R_0603_HandSoldering
- U1, U3: footprint (none) -> SMD_Packages:SOIC-14_N
- U1: renamed from U3; footprint (none) -> SMD_Packages:SOIC-14_N
- U2: footprint (none) -> SMD_Packages:SOIC-8-N
- U3: renamed from U1; footprint (none) -> SMD_Packages:SOIC-14_N
Connections:
- net ~CS_MB: now reaches P2.1 (P1)
- net ~CS_MB: now also U1.2 (O/I); no longer U1.3 (O/I)
- net ~CS: now reaches U2.1 (~CS), U3.2 (O/I)
- net ~CS: now also U1.1 (I/O); no longer U1.4 (I/O)
- net SO_MB: now reaches P2.3 (P3)
- net SO_MB: now also U1.3 (O/I); no longer U1.10 (O/I)
- net SI_MB: now reaches P2.8 (P8)
- net SI_MB: now also U1.9 (O/I); no longer U1.3 (O/I)
- net CLK_MB: now reaches P2.6 (P6), U1.10 (O/I)
- net CLK: now reaches U1.11 (I/O), U2.6 (CLK)
- net CLK: now also U3.10 (O/I); no longer U3.9 (O/I)
- net ~WP: now reaches R2.1, U2.3 (~WP)
- net ~CS_FL: now reaches P1.1 (P1), U3.1 (I/O)
- net SI_FL: now reaches P1.3 (P3)
- net SI_FL: now also U3.4 (I/O); no longer U3.8 (I/O)
- net CLK_FL: now reaches P1.6 (P6)
- net CLK_FL: now also U3.11 (I/O); no longer U3.8 (I/O)
- net SO_FL: now reaches P1.8 (P8)
- net SO_FL: now also U3.8 (I/O); no longer U3.1 (I/O)
- new net EN_FL: J1.1 (Pin_1), U3.12 (ON), U3.13 (ON), U3.5 (ON), U3.6 (ON)
- new net EN_MB: J1.3 (Pin_3), U1.12 (ON), U1.13 (ON), U1.5 (ON), U1.6 (ON)
- new net SI: U1.8 (I/O), U2.5 (SI), U3.9 (O/I)
- new net SO: U1.4 (I/O), U2.2 (SO), U3.3 (O/I)
Changed lines of the file:
@@
 $Comp
 L 4066 U1
-U 2 1 5B0F4DC0
+U 1 1 5B0F4DC0
 P 4050 5050
 F 0 "U1" H 4250 4901 50  0000 C CNN
 F 1 "4066" H 4250 5200 50  0000 C CNN
-F 2 "" H 4050 5050 60  0001 C CNN
+F 2 "SMD_Packages:SOIC-14_N" H 4050 5050 60  0001 C CNN
 F 3 "" H 4050 5050 60  0001 C CNN
-	2    4050 5050
+	1    4050 5050
 	0    1    1    0
 $EndComp
 $Comp
 L 4066 U1
-U 4 1 5B0F4E1D
+U 2 1 5B0F4E1D
 P 5000 5050
 F 0 "U1" H 5200 4901 50  0000 C CNN
 F 1 "4066" H 5200 5200 50  0000 C CNN
-F 2 "" H 5000 5050 60  0001 C CNN
+F 2 "SMD_Packages:SOIC-14_N" H 5000 5050 60  0001 C CNN
 F 3 "" H 5000 5050 60  0001 C CNN
-	4    5000 5050
-	0    1    1    0
-$EndComp
-$Comp
-L 4066 U3
-U 2 1 5B0F4E8A
+	2    5000 5050
+	0    1    1    0
+$EndComp
+$Comp
+L 4066 U1
+U 3 1 5B0F4E8A
 P 6000 5050
-F 0 "U3" H 6200 4901 50  0000 C CNN
+F 0 "U1" H 6200 4901 50  0000 C CNN
 F 1 "4066" H 6200 5200 50  0000 C CNN
-F 2 "" H 6000 5050 60  0001 C CNN
+F 2 "SMD_Packages:SOIC-14_N" H 6000 5050 60  0001 C CNN
 F 3 "" H 6000 5050 60  0001 C CNN
-	2    6000 5050
-	0    1    1    0
-$EndComp
-$Comp
-L 4066 U3
+	3    6000 5050
+	0    1    1    0
+$EndComp
+$Comp
+L 4066 U1
 U 4 1 5B0F4F29
 P 6950 5050
-F 0 "U3" H 7150 4901 50  0000 C CNN
+F 0 "U1" H 7150 4901 50  0000 C CNN
 F 1 "4066" H 7150 5200 50  0000 C CNN
-F 2 "" H 6950 5050 60  0001 C CNN
+F 2 "SMD_Packages:SOIC-14_N" H 6950 5050 60  0001 C CNN
 F 3 "" H 6950 5050 60  0001 C CNN
 	4    6950 5050
@@
 F 0 "U2" H 5350 4350 60  0000 C CNN
 F 1 "25LXX" H 5150 3700 60  0000 C CNN
-F 2 "" H 5050 3900 60  0001 C CNN
+F 2 "SMD_Packages:SOIC-8-N" H 5050 3900 60  0001 C CNN
 F 3 "" H 5050 3900 60  0001 C CNN
 	1    5150 4050
@@
 F 0 "P2" H 5350 6450 50  0000 C CNN
 F 1 "CONN_02X04" H 5350 5950 50  0000 C CNN
-F 2 "" H 5350 5000 50  0000 C CNN
+F 2 "Pin_Headers:Pin_Header_Straight_2x04_Pitch2.54mm" H 5350 5000 50  0001 C CNN
 F 3 "" H 5350 5000 50  0000 C CNN
 	1    5350 6200
@@
 F 0 "P1" H 5350 1650 50  0000 C CNN
 F 1 "CONN_02X04" H 5350 1150 50  0000 C CNN
-F 2 "" H 5350 200 50  0000 C CNN
+F 2 "Pin_Headers:Pin_Header_Straight_2x04_Pitch2.54mm" H 5350 200 50  0001 C CNN
 F 3 "" H 5350 200 50  0000 C CNN
 	1    5350 1400
@@
 F 0 "R3" V 5930 4000 50  0000 C CNN
 F 1 "10k" V 5850 4000 50  0000 C CNN
-F 2 "" V 5780 4000 50  0001 C CNN
+F 2 "Resistors_SMD:R_0603_HandSoldering" V 5780 4000 50  0001 C CNN
 F 3 "" H 5850 4000 50  0001 C CNN
 	1    5850 4000
@@
 F 0 "R2" V 4030 4100 50  0000 C CNN
 F 1 "10k" V 3950 4100 50  0000 C CNN
-F 2 "" V 3880 4100 50  0001 C CNN
+F 2 "Resistors_SMD:R_0603_HandSoldering" V 3880 4100 50  0001 C CNN
 F 3 "" H 3950 4100 50  0001 C CNN
 	1    3950 4100
@@
 $EndComp
 $Comp
-L 4066 U1
+L 4066 U3
 U 1 1 5B0FD800
 P 4050 2900
-F 0 "U1" H 4250 2751 50  0000 C CNN
+F 0 "U3" H 4250 2751 50  0000 C CNN
 F 1 "4066" H 4250 3050 50  0000 C CNN
-F 2 "" H 4050 2900 60  0001 C CNN
+F 2 "SMD_Packages:SOIC-14_N" H 4050 2900 60  0001 C CNN
 F 3 "" H 4050 2900 60  0001 C CNN
 	1    4050 2900
@@
 $EndComp
 $Comp
-L 4066 U1
-U 3 1 5B0FD806
+L 4066 U3
+U 2 1 5B0FD806
 P 5000 2900
-F 0 "U1" H 5200 2751 50  0000 C CNN
+F 0 "U3" H 5200 2751 50  0000 C CNN
 F 1 "4066" H 5200 3050 50  0000 C CNN
-F 2 "" H 5000 2900 60  0001 C CNN
+F 2 "SMD_Packages:SOIC-14_N" H 5000 2900 60  0001 C CNN
 F 3 "" H 5000 2900 60  0001 C CNN
-	3    5000 2900
+	2    5000 2900
 	0    1    1    0
 $EndComp
 $Comp
 L 4066 U3
-U 1 1 5B0FD80C
+U 3 1 5B0FD80C
 P 6000 2900
 F 0 "U3" H 6200 2751 50  0000 C CNN
 F 1 "4066" H 6200 3050 50  0000 C CNN
-F 2 "" H 6000 2900 60  0001 C CNN
+F 2 "SMD_Packages:SOIC-14_N" H 6000 2900 60  0001 C CNN
 F 3 "" H 6000 2900 60  0001 C CNN
-	1    6000 2900
+	3    6000 2900
 	0    1    1    0
 $EndComp
 $Comp
 L 4066 U3
-U 3 1 5B0FD812
+U 4 1 5B0FD812
 P 6950 2900
 F 0 "U3" H 7150 2751 50  0000 C CNN
 F 1 "4066" H 7150 3050 50  0000 C CNN
-F 2 "" H 6950 2900 60  0001 C CNN
+F 2 "SMD_Packages:SOIC-14_N" H 6950 2900 60  0001 C CNN
 F 3 "" H 6950 2900 60  0001 C CNN
-	3    6950 2900
+	4    6950 2900
 	0    1    1    0
 $EndComp
@@
 F 0 "C1" H 6210 4120 50  0000 L CNN
 F 1 "10nF" H 6210 3970 50  0000 L CNN
-F 2 "" H 6200 4050 50  0001 C CNN
+F 2 "Capacitors_SMD:C_0603_HandSoldering" H 6200 4050 50  0001 C CNN
 F 3 "" H 6200 4050 50  0001 C CNN
 	1    6200 4050
@@
 F 0 "C2" H 7810 1820 50  0000 L CNN
 F 1 "10uF" H 7810 1670 50  0000 L CNN
-F 2 "" H 7800 1750 50  0001 C CNN
+F 2 "Capacitors_SMD:C_0603_HandSoldering" H 7800 1750 50  0001 C CNN
 F 3 "" H 7800 1750 50  0001 C CNN
 	1    7800 1750
@@
 F 0 "J2" H 7750 1100 50  0000 C CNN
 F 1 "Conn_01x03_Male" H 7750 700 50  0000 C CNN
-F 2 "" H 7750 900 50  0001 C CNN
+F 2 "Pin_Headers:Pin_Header_Straight_1x03_Pitch2.54mm" H 7750 900 50  0001 C CNN
 F 3 "" H 7750 900 50  0001 C CNN
 	1    7750 900
@@
 F 0 "J1" H 1750 3600 50  0000 C CNN
 F 1 "Conn_01x03_Male" H 1750 3200 50  0000 C CNN
-F 2 "" H 1750 3400 50  0001 C CNN
+F 2 "Pin_Headers:Pin_Header_Straight_1x03_Pitch2.54mm" H 1750 3400 50  0001 C CNN
 F 3 "" H 1750 3400 50  0001 C CNN
 	1    1750 3400
@@
 F 0 "R1" V 2930 3400 50  0000 C CNN
 F 1 "10k" V 2850 3400 50  0000 C CNN
-F 2 "" V 2780 3400 50  0001 C CNN
+F 2 "Resistors_SMD:R_0603_HandSoldering" V 2780 3400 50  0001 C CNN
 F 3 "" H 2850 3400 50  0001 C CNN
 	1    2850 3400
@@
 NoConn ~ 5100 6250
 NoConn ~ 5600 6150
+Text Label 5600 1550 0    60   ~ 0
+SO_FL
+Text Label 5600 1450 0    60   ~ 0
+CLK_FL
+Text Label 5100 1350 2    60   ~ 0
+SI_FL
+Text Label 5100 1250 2    60   ~ 0
+~CS_FL
+Text Label 5600 1250 0    60   ~ 0
+VCC_FL
+Text Label 4900 6050 2    60   ~ 0
+~CS_MB
+Text Label 5600 6050 0    60   ~ 0
+VCC_MB
+Text Label 5000 5600 3    60   ~ 0
+SO_MB
+Text Label 5600 6250 0    60   ~ 0
+CLK_MB
+Text Label 5600 6350 0    60   ~ 0
+SI_MB
 Wire Wire Line
 	5600 4000 5700 4000
@@
 	4050 6050 5100 6050
 Wire Wire Line
-	5000 5350 5000 6150
-Wire Wire Line
-	5000 6150 5100 6150
-Wire Wire Line
 	5600 6250 6950 6250
 Wire Wire Line
@@
 Wire Wire Line
 	4050 1250 4050 2600
-Wire Wire Line
-	6000 1550 6000 2600
 Wire Wire Line
 	6950 1450 6950 2600
@@
 	5600 1450 6950 1450
 Wire Wire Line
-	6000 1550 5600 1550
-Wire Wire Line
 	7200 2900 7300 2900
 Wire Wire Line
@@
 Wire Wire Line
 	4650 2900 4750 2900
+Wire Wire Line
+	5600 1550 6000 1550
+Wire Wire Line
+	6000 1550 6000 2600
+Text Label 2000 3500 0    60   ~ 0
+EN_MB
+Text Label 2000 3300 0    60   ~ 0
+EN_FL
+Wire Wire Line
+	5000 5350 5000 6150
+Wire Wire Line
+	5000 6150 5100 6150
+Text Label 4700 3900 2    60   ~ 0
+~CS
+Text Label 4700 4000 2    60   ~ 0
+SO
+Text Label 4700 4100 2    60   ~ 0
+~WP
+Text Label 5600 3900 0    60   ~ 0
+VCC
+Text Label 5650 4400 0    60   ~ 0
+CLK
+Text Label 5650 4200 0    60   ~ 0
+SI
 $EndSCHEMATC
